File: keypad/keypad.kicad_pcb (KiCad board)
At the start: 2 copper layers, 50 x 58.2 mm, 60 parts, among them J1 NO FIT, P1 GT-USB-7010ASV, Q1 BC807-40LT1G, SW1 TS04-66-70-BK-100-SMT, SW2 TS04-66-70-BK-100-SMT, SW3 NO FIT, SW4 NO FIT, SW5 NO FIT, U1 RP2040, U3 W25Q16JVSSIQ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

Commit message: realign everything
Parts:
- SW4, SW5: footprint Button_Switch_Keyboard:SW_Cherry_MX_1.00u_PCB -> Switch_Keyboard_Cherry_MX:SW_Cherry_MX_PCB_1.00u
- moved SW4 5.72 mm to (95.4, 79.4)
- moved SW5 5.56 mm to (114.6, 79.4)
- moved C19 2.97 mm to (111.4, 70.2)
- moved U5 2.97 mm to (114.6, 70.2)
- moved SW2 2.92 mm to (121.0, 95.0)
- moved C10 2.83 mm to (101.4, 101.0)
- moved C11 2.83 mm to (98.4, 107.0)
- moved C12 2.83 mm to (106.2, 100.0)
- moved C13 2.83 mm to (92.2, 73.4)
- moved C14 2.83 mm to (108.6, 100.0)
- moved C15 2.83 mm to (119.3, 76.5)
- moved C16 2.83 mm to (98.2, 92.8)
- moved C17 2.83 mm to (102.2, 92.0)
- moved C18 2.83 mm to (95.8, 92.2)
- moved C20 2.83 mm to (91.4, 70.2)
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Routing:
- net +3.3V: track 191.7 -> 198.9 mm
- net ADC1: track 45.4 -> 44.6 mm
- net ADC0: track 42.0 -> 41.4 mm
